File: Reset Handler.sch (EAGLE design)
At the start: 13 parts, among them IC1 NE555P, T1 2N222A

Commit message: Finished Reset Handler board.
Parts:
- D1: value 1N4148DO35-7 -> 1N4148
- GPIO1: value RPI_GPIOUPPER -> RPI_GPIO_MALE_OPEN; device connectors:RPI_GPIOUPPER -> connectors:RPI_GPIO_MALE_OPEN
Connections:
- new net N$5: C3.2, IC1.CV
- net GND: no longer C3.2, IC1.CV
Other:
- moved on the sheet: C3
Changed lines of the file:
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@@
 <grid distance="0.1" unitdist="inch" unit="inch" style="lines" multiple="1" display="no" altdistance="0.01" altunitdist="inch" altunit="inch"/>
 <layers>
-<layer number="1" name="Top" color="4" fill="1" visible="no" active="no"/>
-<layer number="16" name="Bottom" color="1" fill="1" visible="no" active="no"/>
-<layer number="17" name="Pads" color="2" fill="1" visible="no" active="no"/>
-<layer number="18" name="Vias" color="2" fill="1" visible="no" active="no"/>
-<layer number="19" name="Unrouted" color="6" fill="1" visible="no" active="no"/>
-<layer number="20" name="Dimension" color="15" fill="1" visible="no" active="no"/>
-<layer number="21" name="tPlace" color="7" fill="1" visible="no" active="no"/>
-<layer number="22" name="bPlace" color="7" fill="1" visible="no" active="no"/>
-<layer number="23" name="tOrigins" color="15" fill="1" visible="no" active="no"/>
-<layer number="24" name="bOrigins" color="15" fill="1" visible="no" active="no"/>
-<layer number="25" name="tNames" color="7" fill="1" visible="no" active="no"/>
-<layer number="26" name="bNames" color="7" fill="1" visible="no" active="no"/>
-<layer number="27" name="tValues" color="7" fill="1" visible="no" active="no"/>
-<layer number="28" name="bValues" color="7" fill="1" visible="no" active="no"/>
+<layer number="1" name="Top" color="4" fill="1" visible="yes" active="no"/>
+<layer number="16" name="Bottom" color="1" fill="1" visible="yes" active="no"/>
+<layer number="17" name="Pads" color="2" fill="1" visible="yes" active="no"/>
+<layer number="18" name="Vias" color="2" fill="1" visible="yes" active="no"/>
+<layer number="19" name="Unrouted" color="6" fill="1" visible="yes" active="no"/>
+<layer number="20" name="Dimension" color="15" fill="1" visible="yes" active="no"/>
+<layer number="21" name="tPlace" color="7" fill="1" visible="yes" active="no"/>
+<layer number="22" name="bPlace" color="7" fill="1" visible="yes" active="no"/>
+<layer number="23" name="tOrigins" color="15" fill="1" visible="yes" active="no"/>
+<layer number="24" name="bOrigins" color="15" fill="1" visible="yes" active="no"/>
+<layer number="25" name="tNames" color="7" fill="1" visible="yes" active="no"/>
+<layer number="26" name="bNames" color="7" fill="1" visible="yes" active="no"/>
+<layer number="27" name="tValues" color="7" fill="1" visible="yes" active="no"/>
+<layer number="28" name="bValues" color="7" fill="1" visible="yes" active="no"/>
 <layer number="29" name="tStop" color="7" fill="3" visible="no" active="no"/>
 <layer number="30" name="bStop" color="7" fill="6" visible="no" active="no"/>
@@
 <layer number="35" name="tGlue" color="7" fill="4" visible="no" active="no"/>
 <layer number="36" name="bGlue" color="7" fill="5" visible="no" active="no"/>
-<layer number="37" name="tTest" color="7" fill="1" visible="no" active="no"/>
-<layer number="38" name="bTest" color="7" fill="1" visible="no" active="no"/>
+<layer number="37" name="tTest" color="7" fill="1" visible="yes" active="no"/>
+<layer number="38" name="bTest" color="7" fill="1" visible="yes" active="no"/>
 <layer number="39" name="tKeepout" color="4" fill="11" visible="no" active="no"/>
 <layer number="40" name="bKeepout" color="1" fill="11" visible="no" active="no"/>
@@
 <layer number="44" name="Drills" color="7" fill="1" visible="no" active="no"/>
 <layer number="45" name="Holes" color="7" fill="1" visible="no" active="no"/>
-<layer number="46" name="Milling" color="3" fill="1" visible="no" active="no"/>
-<layer number="47" name="Measures" color="7" fill="1" visible="no" active="no"/>
-<layer number="48" name="Document" color="7" fill="1" visible="no" active="no"/>
-<layer number="49" name="Reference" color="7" fill="1" visible="no" active="no"/>
-<layer number="51" name="tDocu" color="7" fill="1" visible="no" active="no"/>
-<layer number="52" name="bDocu" color="7" fill="1" visible="no" active="no"/>
+<layer number="46" name="Milling" color="3" fill="1" visible="yes" active="no"/>
+<layer number="47" name="Measures" color="7" fill="1" visible="yes" active="no"/>
+<layer number="48" name="Document" color="7" fill="1" visible="yes" active="no"/>
+<layer number="49" name="Reference" color="7" fill="1" visible="yes" active="no"/>
+<layer number="51" name="tDocu" color="7" fill="1" visible="yes" active="no"/>
+<layer number="52" name="bDocu" color="7" fill="1" visible="yes" active="no"/>
 <layer number="90" name="Modules" color="5" fill="1" visible="yes" active="yes"/>
 <layer number="91" name="Nets" color="2" fill="1" visible="yes" active="yes"/>
@@
 <part name="C3" library="capacitor-wima" deviceset="C" device="10/4" value="0.01uF"/>
 <part name="C2" library="capacitor-wima" deviceset="C" device="10/4" value="0.01uF"/>
-<part name="D1" library="diode" deviceset="1N4148" device="DO35-7"/>
+<part name="D1" library="diode" deviceset="1N4148" device="DO35-7" value="1N4148"/>
 <part name="RESET" library="pinhead" deviceset="PINHD-1X2" device=""/>
-<part name="GPIO1" library="connectors" deviceset="RPI_GPIO*" device="UPPER"/>
+<part name="GPIO1" library="connectors" deviceset="RPI_GPIO*" device="_MALE_OPEN"/>
 <part name="R3" library="te-connectivity" deviceset="OUAZ-*" device="OUAZ-SS-105D" value="5VDC"/>
 </parts>
@@
 </instance>
 <instance part="CT" gate="G$1" x="68.58" y="43.18"/>
-<instance part="C3" gate="G$1" x="20.32" y="50.8" smashed="yes" rot="R180">
-<attribute name="NAME" x="16.764" y="47.625" size="1.778" layer="95" rot="R180"/>
-<attribute name="VALUE" x="19.304" y="57.531" size="1.778" layer="96" rot="R180"/>
+<instance part="C3" gate="G$1" x="20.32" y="43.18" smashed="yes" rot="R180">
+<attribute name="NAME" x="16.764" y="40.005" size="1.778" layer="95" rot="R180"/>
+<attribute name="VALUE" x="19.304" y="49.911" size="1.778" layer="96" rot="R180"/>
 </instance>
 <instance part="C2" gate="G$1" x="10.16" y="66.04" smashed="yes" rot="R270">
@@
 <bus name="UART0_TXD,UART0_RXD,GPIO_4,GPIO_5,GPIO_6,GPIO_12,GPIO_13,GPIO_16,GPIO_17,GPIO_18,GPIO_19,GPIO_20,GPIO_21,GPIO_22,GPIO_23,GPIO_24,GPIO_25,GPIO_26,GPIO_27">
 <segment>
-<wire x1="22.86" y1="22.86" x2="-5.08" y2="22.86" width="0.762" layer="92"/>
-<wire x1="22.86" y1="22.86" x2="22.86" y2="-17.78" width="0.762" layer="92"/>
+<wire x1="20.32" y1="22.86" x2="-5.08" y2="22.86" width="0.762" layer="92"/>
+<wire x1="20.32" y1="22.86" x2="20.32" y2="-17.78" width="0.762" layer="92"/>
 </segment>
 </bus>
@@
 <junction x="12.7" y="88.9"/>
 <wire x1="27.94" y1="88.9" x2="27.94" y2="60.96" width="0.1524" layer="91"/>
-<wire x1="27.94" y1="60.96" x2="30.48" y2="60.96" width="0.1524" layer="91"/>
-<pinref part="IC1" gate="A" pin="R"/>
-<junction x="30.48" y="60.96"/>
 <wire x1="20.32" y1="88.9" x2="27.94" y2="88.9" width="0.1524" layer="91"/>
 <junction x="20.32" y="88.9"/>
@@
 <wire x1="68.58" y1="88.9" x2="83.82" y2="88.9" width="0.1524" layer="91"/>
 <junction x="68.58" y="88.9"/>
+<pinref part="IC1" gate="A" pin="R"/>
+<wire x1="27.94" y1="60.96" x2="30.48" y2="60.96" width="0.1524" layer="91"/>
 </segment>
 <segment>
@@
 <wire x1="5.08" y1="33.02" x2="5.08" y2="48.26" width="0.1524" layer="91"/>
 <wire x1="-10.16" y1="33.02" x2="5.08" y2="33.02" width="0.1524" layer="91"/>
-<pinref part="IC1" gate="A" pin="CV"/>
-<pinref part="C3" gate="G$1" pin="2"/>
-<wire x1="20.32" y1="55.88" x2="30.48" y2="55.88" width="0.1524" layer="91"/>
-<pinref part="C3" gate="G$1" pin="1"/>
-<wire x1="20.32" y1="48.26" x2="20.32" y2="55.88" width="0.1524" layer="91"/>
-<wire x1="20.32" y1="33.02" x2="20.32" y2="48.26" width="0.1524" layer="91"/>
-<junction x="20.32" y="48.26"/>
-<junction x="20.32" y="55.88"/>
 <wire x1="5.08" y1="33.02" x2="20.32" y2="33.02" width="0.1524" layer="91"/>
 <junction x="5.08" y="33.02"/>
+<wire x1="20.32" y1="33.02" x2="27.94" y2="33.02" width="0.1524" layer="91"/>
 <wire x1="27.94" y1="33.02" x2="27.94" y2="50.8" width="0.1524" layer="91"/>
 <pinref part="IC1" gate="A" pin="GND"/>
 <wire x1="27.94" y1="50.8" x2="30.48" y2="50.8" width="0.1524" layer="91"/>
-<wire x1="20.32" y1="33.02" x2="27.94" y2="33.02" width="0.1524" layer="91"/>
-<junction x="20.32" y="33.02"/>
 <wire x1="27.94" y1="33.02" x2="68.58" y2="33.02" width="0.1524" layer="91"/>
 <junction x="27.94" y="33.02"/>
@@
 <pinref part="R3" gate="G$1" pin="COIL2"/>
 <wire x1="137.16" y1="58.42" x2="137.16" y2="71.12" width="0.1524" layer="91"/>
-</segment>
-</net>
-<net name="SPI0_MISO" class="0">
-<segment>
-<wire x1="12.7" y1="7.62" x2="10.16" y2="7.62" width="0.1524" layer="91"/>
+<pinref part="C3" gate="G$1" pin="1"/>
+<wire x1="20.32" y1="40.64" x2="20.32" y2="33.02" width="0.1524" layer="91"/>
+<junction x="20.32" y="33.02"/>
 </segment>
 </net>
@@
 </segment>
 </net>
+<net name="N$5" class="0">
+<segment>
+<pinref part="IC1" gate="A" pin="CV"/>
+<wire x1="20.32" y1="55.88" x2="30.48" y2="55.88" width="0.1524" layer="91"/>
+<pinref part="C3" gate="G$1" pin="2"/>
+<wire x1="20.32" y1="48.26" x2="20.32" y2="55.88" width="0.1524" layer="91"/>
+</segment>
+</net>
